File: TALLER0.brd (EAGLE design)
At the start: 100 x 80 mm, 11 parts, among them IC1 LM741P, J2 1X5, K1 JJM1-12V, T1 2N2222

Commit message: Final PCB
Parts:
- moved POT2 15.5 mm to (12.7, 15.2)
Connections:
- removed net GNDA: IC1.4, J2.2, POT2.A, R1.1, R2.1, T1.1
- removed net N$12: J2.5, K1.NO
- removed net N$13: J2.3, K1.C
- removed net N$2: PH1.2, R1.2, S1.5
- removed net N$4: POT2.S, S1.2
- removed net N$5: IC1.2, S1.1, S1.6
- removed net N$6: IC1.3, S1.3, S1.4
- removed net N$7: IC1.6, R3.2
- removed net N$8: R2.2, R3.1, T1.2
- removed net N$9: D1.A, K1.2, T1.3
- new net V-: IC1.4
- net V+: no longer D1.C, J2.1, K1.1, PH1.1, POT2.E
Changed lines of the file:
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@@
 <elements>
 <element name="IC1" library="opams" package="DIL08" value="LM741P" x="39.37" y="44.45"/>
-<element name="POT2" library="adafruit" package="THUMBWHEELV" value="THUMBPOTV" x="25.4" y="6.35"/>
+<element name="POT2" library="adafruit" package="THUMBWHEELV" value="THUMBPOTV" x="12.7" y="15.24"/>
 <element name="R1" library="adafruit" package="0207/10" value="" x="-13.97" y="-3.81"/>
 <element name="R2" library="adafruit" package="0207/10" value="" x="-13.97" y="-8.89"/>
@@
 </elements>
 <signals>
-<signal name="N$2">
-<contactref element="R1" pad="2"/>
-<contactref element="PH1" pad="2"/>
-<contactref element="S1" pad="5"/>
-<wire x1="-22.7" y1="-27.94" x2="-40.7924" y2="-34.29" width="0" layer="19" extent="1-1"/>
-<wire x1="-8.89" y1="-3.81" x2="-22.7" y2="-27.94" width="0" layer="19" extent="1-1"/>
+<signal name="V+">
+<contactref element="IC1" pad="7"/>
 </signal>
-<signal name="GNDA">
-<contactref element="R1" pad="1"/>
-<contactref element="POT2" pad="A"/>
+<signal name="V-">
 <contactref element="IC1" pad="4"/>
-<contactref element="R2" pad="1"/>
-<contactref element="T1" pad="1"/>
-<contactref element="J2" pad="2"/>
-<wire x1="20.4" y1="6.35" x2="43.18" y2="40.64" width="0" layer="19" extent="1-1"/>
-<wire x1="-19.05" y1="-3.81" x2="20.4" y2="6.35" width="0" layer="19" extent="1-1"/>
-<wire x1="-19.05" y1="-8.89" x2="-19.05" y2="-3.81" width="0" layer="19" extent="1-1"/>
-<wire x1="-16.51" y1="-20.32" x2="-19.05" y2="-8.89" width="0" layer="19" extent="1-1"/>
-<wire x1="-24.44" y1="-41.91" x2="-16.51" y2="-20.32" width="0" layer="19" extent="1-1"/>
-</signal>
-<signal name="N$4">
-<contactref element="S1" pad="2"/>
-<contactref element="POT2" pad="S"/>
-<wire x1="25.4" y1="5.85" x2="-45.5676" y2="-34.29" width="0" layer="19" extent="1-1"/>
-</signal>
-<signal name="N$5">
-<contactref element="S1" pad="1"/>
-<contactref element="IC1" pad="2"/>
-<contactref element="S1" pad="6"/>
-<wire x1="-45.5676" y1="-30.2768" x2="38.1" y2="40.64" width="0" layer="19" extent="1-1"/>
-<wire x1="-40.7924" y1="-38.3032" x2="-45.5676" y2="-30.2768" width="0" layer="19" extent="1-1"/>
-</signal>
-<signal name="N$6">
-<contactref element="S1" pad="4"/>
-<contactref element="IC1" pad="3"/>
-<contactref element="S1" pad="3"/>
-<wire x1="-40.7924" y1="-30.2768" x2="40.64" y2="40.64" width="0" layer="19" extent="1-1"/>
-<wire x1="-45.5676" y1="-38.3032" x2="-40.7924" y2="-30.2768" width="0" layer="19" extent="1-1"/>
-</signal>
-<signal name="V+">
-<contactref element="J2" pad="1"/>
-<contactref element="PH1" pad="1"/>
-<contactref element="POT2" pad="E"/>
-<contactref element="IC1" pad="7"/>
-<contactref element="K1" pad="1"/>
-<contactref element="D1" pad="C"/>
-<wire x1="-20.94" y1="-41.91" x2="-40.64" y2="-48.26" width="0" layer="19" extent="1-1"/>
-<wire x1="-28.1" y1="-27.94" x2="-20.94" y2="-41.91" width="0" layer="19" extent="1-1"/>
-<wire x1="-7.38" y1="-24.21" x2="-28.1" y2="-27.94" width="0" layer="19" extent="1-1"/>
-<wire x1="30.4" y1="6.35" x2="-7.38" y2="-24.21" width="0" layer="19" extent="1-1"/>
-<wire x1="38.1" y1="48.26" x2="30.4" y2="6.35" width="0" layer="19" extent="1-1"/>
-</signal>
-<signal name="N$7">
-<contactref element="IC1" pad="6"/>
-<contactref element="R3" pad="2"/>
-<wire x1="-8.89" y1="-13.97" x2="40.64" y2="48.26" width="0" layer="19" extent="1-1"/>
-</signal>
-<signal name="N$8">
-<contactref element="R3" pad="1"/>
-<contactref element="R2" pad="2"/>
-<contactref element="T1" pad="2"/>
-<wire x1="-19.05" y1="-13.97" x2="-13.97" y2="-20.32" width="0" layer="19" extent="1-1"/>
-<wire x1="-8.89" y1="-8.89" x2="-19.05" y2="-13.97" width="0" layer="19" extent="1-1"/>
-</signal>
-<signal name="N$9">
-<contactref element="T1" pad="3"/>
-<contactref element="K1" pad="2"/>
-<contactref element="D1" pad="A"/>
-<wire x1="-7.38" y1="-34.21" x2="-48.26" y2="-48.26" width="0" layer="19" extent="1-1"/>
-<wire x1="-13.97" y1="-17.78" x2="-7.38" y2="-34.21" width="0" layer="19" extent="1-1"/>
-</signal>
-<signal name="N$12">
-<contactref element="J2" pad="5"/>
-<contactref element="K1" pad="NO"/>
-<wire x1="-17.58" y1="-24.21" x2="-34.94" y2="-41.91" width="0" layer="19" extent="1-1"/>
-</signal>
-<signal name="N$13">
-<contactref element="K1" pad="C"/>
-<contactref element="J2" pad="3"/>
-<wire x1="-4.88" y1="-29.21" x2="-27.94" y2="-41.91" width="0" layer="19" extent="1-1"/>
 </signal>
 </signals>

Commit message: RAS UNI 08/06/2019.
Connections:
- removed net V-: IC1.4
- new net GNDA: IC1.4, J2.2, POT2.A, R1.1, R2.1, T1.1
- new net N$1: PH1.2, R1.2
- new net N$10: D1.A, K1.2, T1.3
- new net N$14: J2.5, K1.NO
- new net N$15: J2.3
- new net N$4: IC1.3, S1.1, S1.6
- new net N$6: IC1.2, S1.3, S1.4
- new net N$7: IC1.6, R3.2
- new net N$8: R2.2, R3.1, T1.2
- net V+: now also D1.C, J2.1, K1.1, PH1.1, POT2.E
Changed lines of the file:
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@@
 <layers>
 <layer number="1" name="Top" color="4" fill="1" visible="yes" active="yes"/>
+<layer number="2" name="Route2" color="1" fill="3" visible="no" active="yes"/>
+<layer number="3" name="Route3" color="4" fill="3" visible="no" active="yes"/>
+<layer number="4" name="Route4" color="1" fill="4" visible="no" active="yes"/>
+<layer number="5" name="Route5" color="4" fill="4" visible="no" active="yes"/>
+<layer number="6" name="Route6" color="1" fill="8" visible="no" active="yes"/>
+<layer number="7" name="Route7" color="4" fill="8" visible="no" active="yes"/>
+<layer number="8" name="Route8" color="1" fill="2" visible="no" active="yes"/>
+<layer number="9" name="Route9" color="4" fill="2" visible="no" active="yes"/>
+<layer number="10" name="Route10" color="1" fill="7" visible="no" active="yes"/>
+<layer number="11" name="Route11" color="4" fill="7" visible="no" active="yes"/>
+<layer number="12" name="Route12" color="1" fill="5" visible="no" active="yes"/>
+<layer number="13" name="Route13" color="4" fill="5" visible="no" active="yes"/>
+<layer number="14" name="Route14" color="1" fill="6" visible="no" active="yes"/>
+<layer number="15" name="Route15" color="4" fill="6" visible="no" active="yes"/>
 <layer number="16" name="Bottom" color="1" fill="1" visible="yes" active="yes"/>
 <layer number="17" name="Pads" color="2" fill="1" visible="yes" active="yes"/>
@@
 <signal name="V+">
 <contactref element="IC1" pad="7"/>
-</signal>
-<signal name="V-">
+<contactref element="PH1" pad="1"/>
+<contactref element="POT2" pad="E"/>
+<contactref element="K1" pad="1"/>
+<contactref element="D1" pad="C"/>
+<contactref element="J2" pad="1"/>
+<wire x1="-20.94" y1="-41.91" x2="-40.64" y2="-48.26" width="0" layer="19" extent="1-1"/>
+<wire x1="-28.1" y1="-27.94" x2="-20.94" y2="-41.91" width="0" layer="19" extent="1-1"/>
+<wire x1="-7.38" y1="-24.21" x2="-28.1" y2="-27.94" width="0" layer="19" extent="1-1"/>
+<wire x1="17.7" y1="15.24" x2="-7.38" y2="-24.21" width="0" layer="19" extent="1-1"/>
+<wire x1="38.1" y1="48.26" x2="17.7" y2="15.24" width="0" layer="19" extent="1-1"/>
+</signal>
+<signal name="N$1">
+<contactref element="R1" pad="2"/>
+<contactref element="PH1" pad="2"/>
+<wire x1="-8.89" y1="-3.81" x2="-22.7" y2="-27.94" width="0" layer="19" extent="1-1"/>
+</signal>
+<signal name="GNDA">
+<contactref element="R1" pad="1"/>
+<contactref element="POT2" pad="A"/>
 <contactref element="IC1" pad="4"/>
+<contactref element="R2" pad="1"/>
+<contactref element="T1" pad="1"/>
+<contactref element="J2" pad="2"/>
+<wire x1="7.7" y1="15.24" x2="43.18" y2="40.64" width="0" layer="19" extent="1-1"/>
+<wire x1="-19.05" y1="-3.81" x2="7.7" y2="15.24" width="0" layer="19" extent="1-1"/>
+<wire x1="-19.05" y1="-8.89" x2="-19.05" y2="-3.81" width="0" layer="19" extent="1-1"/>
+<wire x1="-16.51" y1="-20.32" x2="-19.05" y2="-8.89" width="0" layer="19" extent="1-1"/>
+<wire x1="-24.44" y1="-41.91" x2="-16.51" y2="-20.32" width="0" layer="19" extent="1-1"/>
+</signal>
+<signal name="N$4">
+<contactref element="IC1" pad="3"/>
+<contactref element="S1" pad="1"/>
+<contactref element="S1" pad="6"/>
+<wire x1="-45.5676" y1="-30.2768" x2="40.64" y2="40.64" width="0" layer="19" extent="1-1"/>
+<wire x1="-40.7924" y1="-38.3032" x2="-45.5676" y2="-30.2768" width="0" layer="19" extent="1-1"/>
+</signal>
+<signal name="N$6">
+<contactref element="S1" pad="4"/>
+<contactref element="S1" pad="3"/>
+<contactref element="IC1" pad="2"/>
+<wire x1="-40.7924" y1="-30.2768" x2="-45.5676" y2="-38.3032" width="0" layer="19" extent="1-1"/>
+<wire x1="38.1" y1="40.64" x2="-40.7924" y2="-30.2768" width="0" layer="19" extent="1-1"/>
+</signal>
+<signal name="N$7">
+<contactref element="IC1" pad="6"/>
+<contactref element="R3" pad="2"/>
+<wire x1="-8.89" y1="-13.97" x2="40.64" y2="48.26" width="0" layer="19" extent="1-1"/>
+</signal>
+<signal name="N$8">
+<contactref element="R3" pad="1"/>
+<contactref element="R2" pad="2"/>
+<contactref element="T1" pad="2"/>
+<wire x1="-19.05" y1="-13.97" x2="-13.97" y2="-20.32" width="0" layer="19" extent="1-1"/>
+<wire x1="-8.89" y1="-8.89" x2="-19.05" y2="-13.97" width="0" layer="19" extent="1-1"/>
+</signal>
+<signal name="N$10">
+<contactref element="K1" pad="2"/>
+<contactref element="T1" pad="3"/>
+<contactref element="D1" pad="A"/>
+<wire x1="-7.38" y1="-34.21" x2="-48.26" y2="-48.26" width="0" layer="19" extent="1-1"/>
+<wire x1="-13.97" y1="-17.78" x2="-7.38" y2="-34.21" width="0" layer="19" extent="1-1"/>
+</signal>
+<signal name="N$14">
+<contactref element="K1" pad="NO"/>
+<contactref element="J2" pad="5"/>
+<wire x1="-17.58" y1="-24.21" x2="-34.94" y2="-41.91" width="0" layer="19" extent="1-1"/>
+</signal>
+<signal name="N$15">
+<contactref element="J2" pad="3"/>
 </signal>
 </signals>
