File: TALLER3.brd (EAGLE design)
At the start: 100 x 80 mm, 11 parts, among them IC1 LM741P, J2 1X5, K1 JJM1-12V, T1 2N2222

Commit message: Final PCB
Parts:
- removed S1: (no value), switch:320-938
- added S2: PVA2, switch-misc:PVA2F
- T1: value 2N2222 -> 2N3904; device transistor-neu-to92:TO18 -> transistor:TO92
- moved J2 147.2 mm to (94.0, 40.6), turned to 270 degrees
- moved D1 141.6 mm to (74.9, 27.9)
- moved K1 115.1 mm to (80.0, 40.6)
- moved R3 114.8 mm to (76.2, 57.1), turned to 180 degrees
- moved T1 108.3 mm to (68.6, 49.5), turned to 270 degrees
- moved PH1 95.5 mm to (54.6, 24.1)
- moved R2 88.6 mm to (66.0, 29.2), turned to 90 degrees
- moved R1 63.8 mm to (40.6, 29.2), turned to 270 degrees
- moved POT2 33.2 mm to (29.2, 39.4), turned to 90 degrees
- moved IC1 11.4 mm to (49.5, 39.4)
Connections:
- net GNDA: now also T1.3; no longer T1.1
- net N$2: now also S2.5; no longer S1.5
- net N$4: now also S2.2; no longer S1.2
- net N$5: now also S2.3, S2.4; no longer S1.1, S1.6
- net N$6: now also S2.1, S2.6; no longer S1.3, S1.4
- net N$9: now also T1.1; no longer T1.3
Routing:
- net N$2: track 0.00 -> 162.5 mm
- net V+: track 0.00 -> 152.0 mm
- net GNDA: track 0.00 -> 122.5 mm
- net N$7: track 0.00 -> 49.1 mm
- net N$9: track 0.00 -> 48.1 mm
- net N$5: track 0.00 -> 44.8 mm
- net N$6: track 0.00 -> 42.2 mm
- net N$4: track 0.00 -> 36.5 mm, vias 0 -> 2
- net N$8: track 0.00 -> 34.3 mm
- net N$12: track 0.00 -> 23.1 mm
- net N$13: track 0.00 -> 7.42 mm
- added copper zone on layer 16, net N$1
Other:
- board size 100 x 80 mm -> 77.1 x 49.5 mm
- board text added: "Nombre proyecto"
- board text added: "UNI"

Commit message: RAS UNI 08/06/2019.
Routing:
- net V+: vias 0 -> 1
- net N$9: vias 0 -> 2
- net N$8: vias 0 -> 1
- net GNDA: vias 0 -> 3
Other:
- board text added: "C:/Users/yesse/Desktop/olympus2.bmp"
